File: Hardware/v2-2/Kicad/Bergoz.sch (KiCad schematic (older format))
At the start: 24 parts, among them J3 BERGOZ_02, J4 BERGOZ_01, Q1 BSR14, Q2 BSR14, T2 CMC, T3 CMC, U1 741G74, U12 1G04, U13 1G04, U14 TS5A21366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

Commit message: Update hardware files
Changed lines of the file:
@@
 LIBS:contrib
 LIBS:valves
-LIBS:Controle
 LIBS:CountingPRU_v2-2-cache
 EELAYER 25 0
@@
 $EndComp
 $Comp
-L GND #PWR79
+L GND #PWR070
 U 1 1 59C2E065
 P 4130 3550
-F 0 "#PWR79" H 4130 3300 50  0001 C CNN
+F 0 "#PWR070" H 4130 3300 50  0001 C CNN
 F 1 "GND" H 4130 3400 50  0000 C CNN
 F 2 "" H 4130 3550 50  0000 C CNN
@@
 $EndComp
 $Comp
-L GND #PWR75
+L GND #PWR071
 U 1 1 59C2E27A
 P 3480 3775
-F 0 "#PWR75" H 3480 3525 50  0001 C CNN
+F 0 "#PWR071" H 3480 3525 50  0001 C CNN
 F 1 "GND" H 3480 3625 50  0000 C CNN
 F 2 "" H 3480 3775 50  0000 C CNN
@@
 D-_02
 $Comp
-L +5V #PWR77
+L +5V #PWR072
 U 1 1 59C2EC15
 P 3780 3000
-F 0 "#PWR77" H 3780 2850 50  0001 C CNN
+F 0 "#PWR072" H 3780 2850 50  0001 C CNN
 F 1 "+5V" H 3780 3140 50  0000 C CNN
 F 2 "" H 3780 3000 50  0000 C CNN
@@
 $EndComp
 $Comp
-L GND #PWR80
+L GND #PWR073
 U 1 1 59C2F81B
 P 4135 4700
-F 0 "#PWR80" H 4135 4450 50  0001 C CNN
+F 0 "#PWR073" H 4135 4450 50  0001 C CNN
 F 1 "GND" H 4135 4550 50  0000 C CNN
 F 2 "" H 4135 4700 50  0000 C CNN
@@
 $EndComp
 $Comp
-L GND #PWR76
+L GND #PWR074
 U 1 1 59C2F821
 P 3485 4925
-F 0 "#PWR76" H 3485 4675 50  0001 C CNN
+F 0 "#PWR074" H 3485 4675 50  0001 C CNN
 F 1 "GND" H 3485 4775 50  0000 C CNN
 F 2 "" H 3485 4925 50  0000 C CNN
@@
 D-_01
 $Comp
-L +5V #PWR78
+L +5V #PWR075
 U 1 1 59C2F83D
 P 3785 4150
-F 0 "#PWR78" H 3785 4000 50  0001 C CNN
+F 0 "#PWR075" H 3785 4000 50  0001 C CNN
 F 1 "+5V" H 3785 4290 50  0000 C CNN
 F 2 "" H 3785 4150 50  0000 C CNN
@@
 $EndComp
 $Comp
-L GND #PWR88
+L GND #PWR076
 U 1 1 59C2FF31
 P 9735 3380
-F 0 "#PWR88" H 9735 3130 50  0001 C CNN
+F 0 "#PWR076" H 9735 3130 50  0001 C CNN
 F 1 "GND" H 9735 3230 50  0000 C CNN
 F 2 "" H 9735 3380 50  0000 C CNN
@@
 -5V
 $Comp
-L GND #PWR87
+L GND #PWR077
 U 1 1 59C303F9
 P 9335 4355
-F 0 "#PWR87" H 9335 4105 50  0001 C CNN
+F 0 "#PWR077" H 9335 4105 50  0001 C CNN
 F 1 "GND" H 9335 4205 50  0000 C CNN
 F 2 "" H 9335 4355 50  0000 C CNN
@@
 $EndComp
 $Comp
-L GND #PWR90
+L GND #PWR078
 U 1 1 59C3063D
 P 10960 3380
-F 0 "#PWR90" H 10960 3130 50  0001 C CNN
+F 0 "#PWR078" H 10960 3130 50  0001 C CNN
 F 1 "GND" H 10960 3230 50  0000 C CNN
 F 2 "" H 10960 3380 50  0000 C CNN
@@
 -5V
 $Comp
-L GND #PWR89
+L GND #PWR079
 U 1 1 59C3064A
 P 10560 4355
-F 0 "#PWR89" H 10560 4105 50  0001 C CNN
+F 0 "#PWR079" H 10560 4105 50  0001 C CNN
 F 1 "GND" H 10560 4205 50  0000 C CNN
 F 2 "" H 10560 4355 50  0000 C CNN
@@
 $EndComp
 $Comp
-L GND #PWR84
+L GND #PWR080
 U 1 1 59E9ED81
 P 7730 4555
-F 0 "#PWR84" H 7730 4305 50  0001 C CNN
+F 0 "#PWR080" H 7730 4305 50  0001 C CNN
 F 1 "GND" H 7730 4405 50  0000 C CNN
 F 2 "" H 7730 4555 50  0000 C CNN
@@
 $EndComp
 $Comp
-L GND #PWR86
+L GND #PWR081
 U 1 1 59E9F641
 P 7730 5505
-F 0 "#PWR86" H 7730 5255 50  0001 C CNN
+F 0 "#PWR081" H 7730 5255 50  0001 C CNN
 F 1 "GND" H 7730 5355 50  0000 C CNN
 F 2 "" H 7730 5505 50  0000 C CNN
@@
 BIN_01
 $Comp
-L GND #PWR74
+L GND #PWR082
 U 1 1 59EA0104
 P 3050 5145
-F 0 "#PWR74" H 3050 4895 50  0001 C CNN
+F 0 "#PWR082" H 3050 4895 50  0001 C CNN
 F 1 "GND" H 3050 4995 50  0000 C CNN
 F 2 "" H 3050 5145 50  0000 C CNN
@@
 	3125 3575 3180 3575
 $Comp
-L GND #PWR73
+L GND #PWR083
 U 1 1 59E9F78C
 P 3005 3975
-F 0 "#PWR73" H 3005 3725 50  0001 C CNN
+F 0 "#PWR083" H 3005 3725 50  0001 C CNN
 F 1 "GND" H 3005 3825 50  0000 C CNN
 F 2 "" H 3005 3975 50  0000 C CNN
@@
 	3050 5125 3050 5145
 $Comp
-L +3.3V #PWR72
+L +3.3V #PWR084
 U 1 1 5A1701CA
 P 2630 5450
-F 0 "#PWR72" H 2630 5300 50  0001 C CNN
+F 0 "#PWR084" H 2630 5300 50  0001 C CNN
 F 1 "+3.3V" H 2630 5590 50  0000 C CNN
 F 2 "" H 2630 5450 50  0001 C CNN
@@
 $EndComp
 $Comp
-L +3.3V #PWR82
+L +3.3V #PWR085
 U 1 1 5A170BA8
 P 5735 1350
-F 0 "#PWR82" H 5735 1200 50  0001 C CNN
+F 0 "#PWR085" H 5735 1200 50  0001 C CNN
 F 1 "+3.3V" H 5735 1490 50  0000 C CNN
 F 2 "" H 5735 1350 50  0001 C CNN
@@
 $EndComp
 $Comp
-L +3.3V #PWR81
+L +3.3V #PWR086
 U 1 1 5A17106F
 P 5135 1700
-F 0 "#PWR81" H 5135 1550 50  0001 C CNN
+F 0 "#PWR086" H 5135 1550 50  0001 C CNN
 F 1 "+3.3V" H 5135 1840 50  0000 C CNN
 F 2 "" H 5135 1700 50  0001 C CNN
@@
 $EndComp
 $Comp
-L +3.3V #PWR71
+L +3.3V #PWR087
 U 1 1 5A17144F
-P 2575 1330
-F 0 "#PWR71" H 2575 1180 50  0001 C CNN
-F 1 "+3.3V" H 2575 1470 50  0000 C CNN
-F 2 "" H 2575 1330 50  0001 C CNN
-F 3 "" H 2575 1330 50  0001 C CNN
-	1    2575 1330
-	1    0    0    -1
-$EndComp
-$Comp
-L +3.3V #PWR70
+P 2575 1195
+F 0 "#PWR087" H 2575 1045 50  0001 C CNN
+F 1 "+3.3V" H 2575 1335 50  0000 C CNN
+F 2 "" H 2575 1195 50  0001 C CNN
+F 3 "" H 2575 1195 50  0001 C CNN
+	1    2575 1195
+	1    0    0    -1
+$EndComp
+$Comp
+L +3.3V #PWR088
 U 1 1 5A1718C3
 P 1975 1680
-F 0 "#PWR70" H 1975 1530 50  0001 C CNN
+F 0 "#PWR088" H 1975 1530 50  0001 C CNN
 F 1 "+3.3V" H 1975 1820 50  0000 C CNN
 F 2 "" H 1975 1680 50  0001 C CNN
@@
 	2890 5430 2890 5125
 $Comp
-L +5V #PWR85
+L +5V #PWR089
 U 1 1 5A6F3C34
 P 7730 4955
-F 0 "#PWR85" H 7730 4805 50  0001 C CNN
+F 0 "#PWR089" H 7730 4805 50  0001 C CNN
 F 1 "+5V" H 7730 5095 50  0000 C CNN
 F 2 "" H 7730 4955 50  0000 C CNN
@@
 $EndComp
 $Comp
-L +5V #PWR83
+L +5V #PWR090
 U 1 1 5A6F3F85
 P 7730 4005
-F 0 "#PWR83" H 7730 3855 50  0001 C CNN
+F 0 "#PWR090" H 7730 3855 50  0001 C CNN
 F 1 "+5V" H 7730 4145 50  0000 C CNN
 F 2 "" H 7730 4005 50  0000 C CNN
@@
 Text HLabel 6135 2475 2    60   Output ~ 0
 CLEAR_1
+Text GLabel 9040 4590 3    60   Input ~ 0
++24V
+Wire Wire Line
+	9040 4590 9040 4180
+Wire Wire Line
+	9040 4180 9035 4180
+Text GLabel 9535 4600 3    60   Input ~ 0
+-5V
+Wire Wire Line
+	9535 4180 9535 4600
+Wire Wire Line
+	9435 4180 9435 4600
+Text GLabel 9435 4600 3    60   Input ~ 0
++5V
+$Comp
+L +5V #PWR091
+U 1 1 5AD0A99D
+P 5825 3955
+F 0 "#PWR091" H 5825 3805 50  0001 C CNN
+F 1 "+5V" H 5825 4095 50  0000 C CNN
+F 2 "" H 5825 3955 50  0000 C CNN
+F 3 "" H 5825 3955 50  0000 C CNN
+	1    5825 3955
+	1    0    0    -1
+$EndComp
+Wire Wire Line
+	5825 3955 5825 4005
+Wire Wire Line
+	5825 4005 6130 4005
+Text HLabel 7930 4180 2    60   Input ~ 0
+CH1
+Text HLabel 7930 4405 2    60   Input ~ 0
+CH2
+Text HLabel 7935 5130 2    60   Input ~ 0
+CH3
+Text HLabel 7935 5355 2    60   Input ~ 0
+CH4
+Wire Wire Line
+	7730 5355 7935 5355
+Wire Wire Line
+	7935 5130 7730 5130
+Wire Wire Line
+	7930 4405 7730 4405
+Wire Wire Line
+	7730 4180 7930 4180
+Text GLabel 2730 1260 2    60   Input ~ 0
++3.3V
+Wire Wire Line
+	2575 1195 2575 1330
+Wire Wire Line
+	2730 1260 2575 1260
+Connection ~ 2575 1260
 $EndSCHEMATC
