File: Hardware/v2-3/Kicad/CountingPRU_v2-3.kicad_pcb (KiCad board)
At the start: 2 copper layers, 160 x 100 mm, 94 parts, among them J1 BBB, J2 IN_ETHERNET, J3 BERGOZ_02, J4 BERGOZ_01, P1 LNLS, P2 LNLS, Q1 BSR14, Q2 BSR14, Q3 BSR14, T1 Module-XFRMR-POE, T2 CMC, T3 CMC, U1 741G74, U10 1G125, U11 1G125, U12 1G04, U13 1G04, U14 TS5A21366, U15 TS5A21366, U16 Ag9205, U17 VIBLSD1-S5-S5-DIP, U18 MEV1D0512DC, U19 1G08, U2 741G74, U20 TS5A21366, U21 74LS123, U22 1G08, U23 741G74, U24 741G74, U25 1G125, U26 1G125, U3 741G74, U4 741G74, U5 741G74, U6 741G74, U7 1G04, U8 1G125, U9 1G125

Commit message: Config pins for kernel 4.14 added
Parts:
- P1: value LNLS -> LNLS 1
- P2: value LNLS -> LNLS 2
Connections:
- Beagle1 pad B26: Net-(Beagle1-PadB26) -> /LED
- Beagle1 pad B8: /LED -> Net-(Beagle1-PadB8)
- U20 pad 1: +5V -> /HardReset_BBB/HARD_RST
- U20 pad 2: /HardReset_BBB/pontoRST -> GND
- U20 pad 4: Net-(U20-Pad4) -> GND
- U20 pad 6: GND -> Net-(U20-Pad6)
- U20 pad 7: GND -> /HardReset_BBB/pontoRST
- U20 pad 8: /HardReset_BBB/HARD_RST -> +5V
Routing:
- net /LED: track 100.7 -> 123.9 mm
- net +5V: track 719.3 -> 728.4 mm
- net GND: track 243.5 -> 240.1 mm
- net /HardReset_BBB/HARD_RST: track 3.80 -> 5.24 mm

Commit message: Updating v2-3 hardware files
Parts:
- JP1: value HR -> HardReset
- U21: value 74LS123 -> 74HC123
Connections:
- Beagle1 pad B26: /LED -> Net-(Beagle1-PadB26)
- Beagle1 pad B28: Net-(Beagle1-PadB28) -> /LED
Routing:
- net /LED: track 123.9 -> 126.4 mm
Other:
- board text added: "CountingPRU v2.3 Junho/2018 Grupo de Controle Patricia Nallin Robert Polli"
- board text removed: "CountingPRU v2.2 Abril/2018 Grupo de Controle Patricia Nallin Robert Polli"
