File: Hardware/v2-3/Kicad/CountingPRU_v2-3.sch (KiCad schematic (older format))
At the start: 33 parts, among them J1 BBB, J2 IN_ETHERNET, P1 LNLS, P2 LNLS, Q3 BSR14, U10 1G125, U11 1G125, U23 741G74, U24 741G74, U25 1G125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

Commit message: Updating v2-3 hardware files
Parts:
- JP1: value HR -> HardReset
- P1: value LNLS -> LNLS 1
- P2: value LNLS -> LNLS 2
Connections:
- net LED: now also Beagle1.B28; no longer Beagle1.B26
Changed lines of the file:
@@
 LIBS:contrib
 LIBS:valves
+LIBS:Controle
 LIBS:CountingPRU_v2-3-cache
 EELAYER 25 0
@@
 P 10110 2670
 F 0 "P2" H 10110 3120 50  0000 C CNN
-F 1 "LNLS" V 10110 2670 50  0000 C CNN
+F 1 "LNLS 2" V 10110 2670 50  0000 C CNN
 F 2 "Pin_Headers:Pin_Header_Angled_2x08_Pitch1.27mm" H 10110 1470 50  0001 C CNN
 F 3 "" H 10110 1470 50  0000 C CNN
@@
 NoConn ~ 7375 5175
 NoConn ~ 7875 4375
-NoConn ~ 7875 5375
+NoConn ~ 7875 5275
 NoConn ~ 7875 5475
 NoConn ~ 7875 5575
@@
 Text Label 3780 1665 2    60   ~ 0
 LED
-Text Label 7875 5275 0    60   ~ 0
+Text Label 7875 5375 0    60   ~ 0
 LED
 $Comp
@@
 P 8250 2645
 F 0 "P1" H 8250 3095 50  0000 C CNN
-F 1 "LNLS" V 8250 2645 50  0000 C CNN
+F 1 "LNLS 1" V 8250 2645 50  0000 C CNN
 F 2 "Pin_Headers:Pin_Header_Angled_2x08_Pitch1.27mm" H 8250 1445 50  0001 C CNN
 F 3 "" H 8250 1445 50  0000 C CNN
@@
 P 5800 1075
 F 0 "JP1" H 5800 1155 50  0000 C CNN
-F 1 "HR" H 5810 1015 50  0001 C CNN
+F 1 "HardReset" H 5810 1015 50  0001 C CNN
 F 2 "Pin_Headers:Pin_Header_Straight_1x02_Pitch2.54mm" H 5800 1075 50  0001 C CNN
 F 3 "" H 5800 1075 50  0000 C CNN
