File: Hardware/v2-3/Kicad/HardReset_BBB.sch (KiCad schematic (older format))
At the start: 17 parts, among them U19 1G08, U20 TS5A21366, U21 74LS123, U22 1G08

Commit message: Updating v2-3 hardware files
Parts:
- U21: value 74LS123 -> 74HC123
Changed lines of the file:
@@
 LIBS:contrib
 LIBS:valves
+LIBS:Controle
 LIBS:CountingPRU_v2-3-cache
 EELAYER 25 0
@@
 P 3450 3525
 F 0 "U21" H 3450 3475 50  0000 C CNN
-F 1 "74LS123" H 3450 3375 50  0000 C CNN
+F 1 "74HC123" H 3450 3375 50  0000 C CNN
 F 2 "Housings_SOIC:SOIC-16_3.9x9.9mm_Pitch1.27mm" H 3450 3525 50  0001 C CNN
 F 3 "" H 3450 3525 50  0000 C CNN
@@
 P 5900 3575
 F 0 "U21" H 5900 3525 50  0000 C CNN
-F 1 "74LS123" H 5900 3425 50  0000 C CNN
+F 1 "74HC123" H 5900 3425 50  0000 C CNN
 F 2 "Housings_SOIC:SOIC-16_3.9x9.9mm_Pitch1.27mm" H 5900 3575 50  0001 C CNN
 F 3 "" H 5900 3575 50  0000 C CNN
